File: schematic/qiroll.kicad_sch (KiCad schematic)
At the start: 91 parts, among them J1 Battery connector, J2 Motor connector, J3 USB_B_Micro, Q1 HYG015N04LS1C2, Q2 HYG015N04LS1C2, Q3 HYG015N04LS1C2, Q4 HYG015N04LS1C2, Q5 HYG015N04LS1C2, Q6 HYG015N04LS1C2, Q7 HYG015N04LS1C2, U1 APM32F407RGT6, U2 ESP32-C3, U3 FD6288T, U4 INA181, U5 INA181, Y1 40 MHz

Commit message: Finished schematic
Signed-off-by: Michael Niewöhner <foss@mniewoehner.de>
Parts:
- removed C26: C, symbol Device:C
- removed D8: D, symbol Device:D
- removed R16: 10k, symbol Device:R
- removed TP14: 5V, symbol Connector:TestPoint
- added C28, C29, C30, C31, C32, C33, C34, C35, C36, C37, C38, C39, C40, C41, C42, C43, C44, C45, C46, C47, C48, C49, C50, C51, C52, C53, C54, C55, C56, C57, C58, C59, C60, C61, C62: C, symbol Device:C
- added D10, D11, D12, D13: D, symbol Device:D
- added D9: RB160MM-60T, symbol Device:D
- added F2: SMD0805B010TF 0.1A, symbol Device:Polyfuse
- added L2, L3, L4: L, symbol Device:L
- added R25, R44, R45, R46, R47: 10k, symbol Device:R
- added R26, R27: 10, symbol Device:R
- added R28: 39k, symbol Device:R
- added R29: 2.2k, symbol Device:R
- added R30, R31, R32, R33, R34, R35, R36, R37: R, symbol Device:R
- added R38, R39, R40: 2k, symbol Device:R
- added R41, R42, R43: 40k, symbol Device:R
- added TP10: 5V, symbol Connector:TestPoint
- added U6, U7: LP2985-3.3, Package_TO_SOT_SMD:SOT-23-5, symbol Regulator_Linear:LP2985-3.3
- added U8, U9: maybe LMR14006/ME3116, Package_TO_SOT_SMD:SOT-23-6, symbol Regulator_Switching:LMR14206
- added Y2: 8 MHz, symbol Device:Crystal_GND2
- R14: value 4.7k -> 10k
- R17: value 10k -> 8k
Connections:
- net E32G0 is gone; now on net SW_START: U2.4 (XTAL_32K_P/ADC1_CH0)
- net E32G1 is gone; now on net USB_ID: U2.5 (XTAL_32K_N/ADC1_CH1)
- net VS1 is gone; now on net BLDC1: C19.2, U3.18 (VS1)
- net VS2 is gone; now on net BLDC2: C20.2, U3.15 (VS2)
- net VS3 is gone; now on net BLDC3: C21.2, U3.12 (VS3)
- net +3.3V-1: now also C52.1, C53.1, C54.1, C55.1, C56.1, C57.1, R45.1, R47.1, U7.5 (VOUT)
- net +3.3V-2: now also R17.1, U1.1 (VBAT), U1.19 (VDD), U1.32 (VDD), U1.48 (VDD), U1.64 (VDD), C45.1, C46.1, C47.1, C48.1, C49.1, C60.1, C61.1, L2.1, U6.5 (VOUT)
- net +37.5V: now also D10.2 (A), R28.1
- net +4.7V: now also C40.1, F2.2, L4.2, R36.2, U6.1 (VIN), U7.1 (VIN), U7.3 (ON/~{OFF})
- net +5V: now also C39.1, C58.1, C59.1, L3.2, R33.2, TP10.1
- net BLDC1: now also R41.1
- net BLDC2: now also R42.1
- net BLDC3: now also R43.1
- net BLDC_NTCP: now also U1.8 (PC0), C44.1, R44.1
- net CUR1: now also U1.27 (PB1), R26.1; no longer U4.1
- net CUR3: now also U1.26 (PB0), R27.1; no longer U5.1
- net GND: now also U1.12 (VSSA), U1.18 (VSS), U1.60 (BOOT0), U1.63 (VSS), C28.2, C29.1, C30.1, C31.2, C32.2, C33.2, C34.2, C37.2, C38.2, C39.2, C40.2, C41.2, C42.2, C43.2, C44.2, C45.2, C46.2, C47.2, C48.2, C49.2, C50.2, C51.2, C52.2, C53.2, C54.2, C55.2, C56.2, C57.2, C58.2, C59.2, C60.2, C61.2, C62.2, D11.2 (A), D12.2 (A), R25.2, R29.2, R30.1, R31.1, R35.1, R37.1, R38.2, R39.2, R40.2, R44.2, U6.2 (GND), U7.2 (GND), U8.2 (GND), U9.2 (GND), Y2.2
- net HIN1: now also U1.43 (PA10)
- net HIN2: now also U1.42 (PA9)
- net HIN3: now also U1.41 (PA8)
- net LIN1: now also U1.36 (PB15)
- net LIN2: now also U1.35 (PB14)
- net LIN3: now also U1.34 (PB13)
- net SW_MODE: now also U2.8 (GPIO3/ADC1_CH3); no longer J3.3 (D+)
- net SW_START: no longer J3.2 (D-)
- net USB_ID: no longer D3.1 (K), J3.4 (ID), R18.2
- net at U2.30 (XTAL_P), Y1.1: now also C50.1
- net at U2.29 (XTAL_N), Y1.3: now also C51.1
- net ESP_G5: now reaches U2.10 (MTDI/GPIO5/ADC2_CH0)
- net ESP_G5: now also U1.20 (PA4), U1.30 (PB11), U1.37 (PC6), R45.2
- net VR2EN: now reaches U2.12 (MTCK/GPIO6)
- net VR2EN: now also U6.3 (ON/~{OFF})
- net ESP_G4: now reaches U2.9 (MTMS/GPIO4/ADC1_CH4)
- net ESP_G4: now also U1.23 (PA7), U1.29 (PB10), U1.38 (PC7), R46.2
- net at J3.1 (VBUS): now also D9.1 (K)
- net at R17.2: now also U1.17 (PA3), C31.1, R25.1
- net at D2.1 (K): now also J3.3 (D+)
- net BAT: now reaches U1.10 (PC2)
- net BAT: now also C43.1, R28.2, R29.1
- net at U1.13 (VDDA): now also L2.2
- net BLDC1_IN: now reaches U1.14 (PA0)
- net BLDC1_IN: now also R38.1, R41.2
- net BLDC2_IN: now reaches U1.15 (PA1)
- net BLDC2_IN: now also R39.1, R42.2
- net BLDC3_IN: now reaches U1.16 (PA2)
- net BLDC3_IN: now also R40.1, R43.2
- net at U1.31 (VCAP_1): now also C29.2
- net at U1.47 (VCAP_2): now also C30.2
- net at U1.5 (PH0): now also Y2.1
- net EN5V: now reaches U1.51 (PC10)
- net EN5V: now also R32.2
- net at U1.6 (PH1): now also Y2.3
- net at U1.7 (NRST): now also C28.1
- net at D1.2 (A), R10.2: now also C32.1
- net E32EN: no longer names the net of C23.1, R12.2, TP7.1, U2.7 (CHIP_EN)
- net E32G3 renamed ESP_G3
- net ESP_G3: now also R47.2; no longer R14.2, U2.8 (GPIO3/ADC1_CH3)
- net ESP32_GPIO1 renamed ESP_G1
- new net: C35.2, D11.1 (K), L3.1, U8.6 (SW)
- new net: C41.1, C42.1, D10.1 (K), R34.2, U8.5 (VIN), U9.5 (VIN)
- new net: D3.1 (K), J3.4 (ID), R18.2
- new net: C33.1, R34.1, R35.2, U9.4 (~{SHDN})
- new net: C36.1, U9.1 (CB)
- new net: C37.1, R36.1, R37.2, U9.3 (FB)
- new net: C36.2, D12.1 (K), L4.1, U9.6 (SW)
- new net: D9.2 (A), F2.1
- new net: R27.2, U5.1
- new net: C34.1, R31.2, R32.1, U8.4 (~{SHDN})
- new net: D13.1 (K), J3.2 (D-)
- new net: C38.1, R30.2, R33.1, U8.3 (FB)
- new net: R26.2, U4.1
- new net: C35.1, U8.1 (CB)
- new net +3.3V-3: R46.1
- new net ESP_G0: C62.1, D13.2 (A), R14.2
- no-connect marks 13 -> 38
Other:
- note removed: "NOT FINISHED YET!"
- note removed: "Note: schematic is incomplete; I left out most caps and VREG circuit details since there is nothing special and they are not needed for understanding the circuit"
- note removed: "VREG Buck 5V (unknown model)"
- note removed: "VREG Buck probably 4.7V/5V (unknown model)"
- note removed: "VREG LDO 3.3V LP2985"
- moved on the sheet: C1, C10, C11, C12, C13, C14, C15, C16, C17, C18, C19, C2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

Commit message: schematic: label USB+/- testpads and correct ESP_G4 pull-up voltage
Signed-off-by: Michael Niewöhner <foss@mniewoehner.de>
Parts:
- TP6: value TestPoint -> USBD+
- TP8: value TestPoint -> USBD-
Connections:
- net +3.3V-3 is gone; now on net +3.3V-2: R46.1
Other:
- note added: "TP6 USBD+"
- note added: "TP8 USBD-"
- note removed: "TP6 XXX"
- note removed: "TP8 XXX"
- moved on the sheet: C29, C30
Changed lines of the file:
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@@
 	)
 	(junction
-		(at 199.39 273.05)
+		(at 199.39 265.43)
 		(diameter 0)
 		(color 0 0 0 0)
@@
 	(wire
 		(pts
-			(xy 196.85 273.05) (xy 199.39 273.05)
+			(xy 196.85 265.43) (xy 199.39 265.43)
 		)
 		(stroke
@@
 	(wire
 		(pts
-			(xy 201.93 251.46) (xy 201.93 265.43)
+			(xy 201.93 251.46) (xy 201.93 257.81)
 		)
 		(stroke
@@
 	(wire
 		(pts
-			(xy 196.85 248.92) (xy 196.85 265.43)
+			(xy 196.85 248.92) (xy 196.85 257.81)
 		)
 		(stroke
@@
 	(wire
 		(pts
-			(xy 199.39 273.05) (xy 201.93 273.05)
+			(xy 199.39 265.43) (xy 201.93 265.43)
 		)
 		(stroke
@@
 	(wire
 		(pts
+			(xy 199.39 266.7) (xy 199.39 265.43)
+		)
+		(stroke
+			(width 0)
+			(type default)
+		)
+	)
+	(wire
+		(pts
 			(xy 224.79 271.78) (xy 224.79 273.05)
 		)
@@
 		)
 	)
-	(text "TP8\nXXX"
+	(text "TP8\nUSBD-"
 		(exclude_from_sim no)
 		(at 107.442 256.794 0)
@@
 		)
 	)
-	(text "TP6\nXXX"
+	(text "TP6\nUSBD+"
 		(exclude_from_sim no)
 		(at 107.442 252.984 0)
@@
 			)
 		)
-		(property "Value" "TestPoint"
+		(property "Value" "USBD-"
 			(at 252.222 210.82 90)
 			(effects
@@
 		(on_board yes)
 		(dnp no)
-		(fields_autoplaced yes)
 		(property "Reference" "#PWR074"
 			(at 273.05 236.22 0)
@@
 			)
 		)
-		(property "Value" "+3.3V-3"
-			(at 273.05 227.33 0)
+		(property "Value" "+3.3V-2"
+			(at 268.986 228.346 0)
 			(effects
 				(font
 					(size 1.27 1.27)
 				)
+				(justify left)
 			)
 		)
@@
 	(symbol
 		(lib_id "Device:C")
-		(at 196.85 269.24 180)
+		(at 196.85 261.62 180)
 		(unit 1)
 		(exclude_from_sim no)
@@
 		(dnp no)
 		(property "Reference" "C29"
-			(at 193.04 268.478 0)
+			(at 193.04 260.858 0)
 			(effects
 				(font
@@
 		)
 		(property "Value" "C"
-			(at 193.04 271.018 0)
+			(at 193.04 263.398 0)
 			(effects
 				(font
@@
 		)
 		(property "Footprint" ""
-			(at 195.8848 265.43 0)
+			(at 195.8848 257.81 0)
 			(effects
 				(font
@@
 		)
 		(property "Datasheet" "~"
-			(at 196.85 269.24 0)
+			(at 196.85 261.62 0)
 			(effects
 				(font
@@
 		)
 		(property "Description" "Unpolarized capacitor"
-			(at 196.85 269.24 0)
+			(at 196.85 261.62 0)
 			(effects
 				(font
@@
 			)
 		)
-		(property "Value" "TestPoint"
+		(property "Value" "USBD+"
 			(at 252.222 213.36 90)
 			(effects
@@
 	(symbol
 		(lib_id "power:GND")
-		(at 199.39 273.05 0)
+		(at 199.39 266.7 0)
 		(unit 1)
 		(exclude_from_sim no)
@@
 		(fields_autoplaced yes)
 		(property "Reference" "#PWR061"
-			(at 199.39 279.4 0)
+			(at 199.39 273.05 0)
 			(effects
 				(font
@@
 		)
 		(property "Value" "GND"
-			(at 199.39 278.384 0)
+			(at 199.39 272.034 0)
 			(effects
 				(font
@@
 		)
 		(property "Footprint" ""
-			(at 199.39 273.05 0)
+			(at 199.39 266.7 0)
 			(effects
 				(font
@@
 		)
 		(property "Datasheet" ""
-			(at 199.39 273.05 0)
+			(at 199.39 266.7 0)
 			(effects
 				(font
@@
 		)
 		(property "Description" "Power symbol creates a global label with name \"GND\" , ground"
-			(at 199.39 273.05 0)
+			(at 199.39 266.7 0)
 			(effects
 				(font
@@
 	(symbol
 		(lib_id "Device:C")
-		(at 201.93 269.24 0)
+		(at 201.93 261.62 0)
 		(mirror x)
 		(unit 1)
@@
 		(dnp no)
 		(property "Reference" "C30"
-			(at 204.978 268.224 0)
+			(at 204.978 260.604 0)
 			(effects
 				(font
@@
 		)
 		(property "Value" "C"
-			(at 204.978 270.764 0)
+			(at 204.978 263.144 0)
 			(effects
 				(font
@@
 		)
 		(property "Footprint" ""
-			(at 202.8952 265.43 0)
+			(at 202.8952 257.81 0)
 			(effects
 				(font
@@
 		)
 		(property "Datasheet" "~"
-			(at 201.93 269.24 0)
+			(at 201.93 261.62 0)
 			(effects
 				(font
@@
 		)
 		(property "Description" "Unpolarized capacitor"
-			(at 201.93 269.24 0)
+			(at 201.93 261.62 0)
 			(effects
 				(font

Commit message: schematic: correct switch connections
Signed-off-by: Michael Niewöhner <foss@mniewoehner.de>
Connections:
- net ESP_G1 is gone; now on net SW_START: C25.1, D3.2 (A), R15.2, R18.1
- net ESP_G3 is gone; now on net SW_MODE: C24.1, D2.2 (A), R47.2
- net USB_ID is gone; now on net SW_START: U2.5 (XTAL_32K_N/ADC1_CH1)
- net ESP_G0: now also U2.4 (XTAL_32K_P/ADC1_CH0)
- net SW_START: no longer U2.4 (XTAL_32K_P/ADC1_CH0)
Changed lines of the file:
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@@
 		)
 	)
-	(label "ESP_G1"
+	(label "SW_START"
 		(at 166.37 46.99 0)
 		(fields_autoplaced yes)
@@
 		)
 	)
-	(label "ESP_G3"
+	(label "SW_MODE"
 		(at 166.37 34.29 0)
 		(fields_autoplaced yes)
@@
 		)
 	)
-	(label "SW_START"
+	(label "ESP_G0"
 		(at 260.35 116.84 180)
 		(fields_autoplaced yes)
@@
 		)
 	)
-	(label "USB_ID"
+	(label "SW_START"
 		(at 260.35 119.38 180)
 		(fields_autoplaced yes)

Commit message: schematic: PA3 is connected to NTC, not resistor
Signed-off-by: Michael Niewöhner <foss@mniewoehner.de>
Parts:
- removed R17: 8k, symbol Device:R
- added TH1: Thermistor_NTC 10k, symbol Device:Thermistor_NTC
Connections:
- net +3.3V-2: now also TH1.1
- net at C31.1, R25.1, U1.17 (PA3): now also TH1.2
Changed lines of the file:
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@@
-	)
-	(symbol
-		(lib_id "Device:R")
-		(at 273.05 186.69 0)
-		(unit 1)
-		(exclude_from_sim no)
-		(in_bom yes)
-		(on_board yes)
-		(dnp no)
-		(property "Reference" "R17"
-			(at 275.59 185.4199 0)
-			(effects
-				(font
-					(size 1.27 1.27)
-				)
-				(justify left)
-			)
-		)
-		(property "Value" "8k"
-			(at 275.59 187.9599 0)
-			(effects
-				(font
-					(size 1.27 1.27)
-				)
-				(justify left)
-			)
-		)
-		(property "Footprint" ""
-			(at 271.272 186.69 90)
-			(effects
-				(font
-					(size 1.27 1.27)
-				)
-				(hide yes)
-			)
-		)
-		(property "Datasheet" "~"
-			(at 273.05 186.69 0)
-			(effects
-				(font
-					(size 1.27 1.27)
-				)
-				(hide yes)
-			)
-		)
-		(property "Description" "Resistor"
-			(at 273.05 186.69 0)
-			(effects
-				(font
-					(size 1.27 1.27)
-				)
-				(hide yes)
-			)
-		)
-		(pin "2"
-		)
-		(pin "1"
-		)
-		(instances
-			(project "qiroll"
-				(path "/f3a3ff6d-cb1b-4dbd-b913-c8be24018339"
-					(reference "R17")
-					(unit 1)
-				)
-			)
-		)
 	)
 	(symbol
@@
 					(unit 1)
 				)
+			)
+		)
+	)
+	(symbol
+		(lib_id "Device:Thermistor_NTC")
+		(at 273.05 186.69 0)
+		(unit 1)
+		(exclude_from_sim no)
+		(in_bom yes)
+		(on_board yes)
+		(dnp no)
+		(fields_autoplaced yes)
+		(property "Reference" "TH1"
+			(at 275.59 185.7374 0)
+			(effects
+				(font
+					(size 1.27 1.27)
+				)
+				(justify left)
+			)
+		)
+		(property "Value" "Thermistor_NTC 10k"
+			(at 275.59 188.2774 0)
+			(effects
+				(font
+					(size 1.27 1.27)
+				)
+				(justify left)
+			)
+		)
+		(property "Footprint" ""
+			(at 273.05 185.42 0)
+			(effects
+				(font
+					(size 1.27 1.27)
+				)
+				(hide yes)
+			)
+		)
+		(property "Datasheet" "~"
+			(at 273.05 185.42 0)
+			(effects
+				(font
+					(size 1.27 1.27)
+				)
+				(hide yes)
+			)
+		)
+		(property "Description" "Temperature dependent resistor, negative temperature coefficient"
+			(at 273.05 186.69 0)
+			(effects
+				(font
+					(size 1.27 1.27)
+				)
+				(hide yes)
+			)
+		)
+		(pin "1"
+		)
+		(pin "2"
+		)
+		(instances
+			(project "qiroll"
+				(path "/f3a3ff6d-cb1b-4dbd-b913-c8be24018339"
+					(reference "TH1")
+					(unit 1)
+				)

Commit message: schematic: correct buttons once again
Signed-off-by: Michael Niewöhner <foss@mniewoehner.de>
Connections:
- net ESP_G0 is gone; now on net SW_START: C62.1, D13.2 (A), R14.2, U2.4 (XTAL_32K_P/ADC1_CH0)
- net SW_START: no longer C25.1, D3.2 (A), R15.2, R18.1, U2.5 (XTAL_32K_N/ADC1_CH1)
- new net ESP_G1: C25.1, D3.2 (A), R15.2, R18.1, U2.5 (XTAL_32K_N/ADC1_CH1)
Changed lines of the file:
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@@
 		)
 	)
-	(label "SW_START"
+	(label "ESP_G1"
 		(at 166.37 46.99 0)
 		(fields_autoplaced yes)
@@
 		)
 	)
-	(label "ESP_G0"
+	(label "SW_START"
 		(at 260.35 116.84 180)
 		(fields_autoplaced yes)
@@
 		)
 	)
-	(label "SW_START"
+	(label "ESP_G1"
 		(at 260.35 119.38 180)
 		(fields_autoplaced yes)
@@
 		)
 	)
-	(label "ESP_G0"
+	(label "SW_START"
 		(at 166.37 40.64 0)
 		(fields_autoplaced yes)
